Commit message: added new STL files and fixed URDF so code compiles

File: irb1600id.urdf (robot description, URDF)
Before this commit: robot abb_irb1600id, 8 links, 7 joints
Links:
- link base_link: geometry collision mesh filename=meshes/irb1600id/collision/base_link.stl; visual mesh filename=meshes/irb1600id/visual/base_link.stl
- link link_1: mass None -> 350; geometry collision mesh filename=meshes/irb1600id/collision/link_1.stl; visual mesh filename=meshes/irb1600id/visual/link_1.stl
- link link_2: mass None -> 300; geometry collision mesh filename=meshes/irb1600id/collision/link_2_whole.stl; visual mesh filename=meshes/irb1600id/visual/link_2.stl
- link link_3: mass None -> 200; geometry collision mesh filename=meshes/irb1600id/collision/link_3.stl; visual mesh filename=meshes/irb1600id/visual/link_3.stl
- link link_4: mass None -> 70; geometry collision mesh filename=meshes/irb1600id/collision/link_4.stl; visual mesh filename=meshes/irb1600id/visual/link_4.stl
- link link_5: mass None -> 20; geometry collision mesh filename=meshes/irb1600id/collision/link_5.stl; visual mesh filename=meshes/irb1600id/visual/link_5.stl
- link link_6: mass None -> 5; geometry collision mesh filename=meshes/irb1600id/collision/link_6.stl; visual mesh filename=meshes/irb1600id/visual/link_6.stl
